Commit message: Updated jupyter notebook test code

File: src/res/flyhopper_mockup/urdf_5kg/flyhopper_mockup.urdf (robot description, URDF)
Before this commit: robot flyhopper_mockup, 3 links, 2 joints
Links:
- link base_link: mass 10 -> 5; geometry collision mesh filename=package://../res/flyhopper_mockup/meshes/base_link.STL; visual mesh filename=package://../res/flyhopper_mockup/meshes/base_link.STL
