Commit message: PID control of leg links working

File: src/res/flyhopper_mockup/urdf/flyhopper_mockup.urdf (robot description, URDF)
Before this commit: robot flyhopper_mockup, 3 links, 2 joints
Links:
- link Link 1: mass 0.624823001646925 -> 0.1
- link Link 2: mass 0.624823001646924 -> 0.1
- link base_link: mass 4.12611894583318 -> 10
Joints:
- joint Joint 1: origin xyz=-0.25981 0 -0.15 rpy=3.1416 0.5236 3.1416 -> xyz=0 0 0 rpy=3.1416 0.5236 3.1416
- joint Joint 2: origin xyz=-0.15 0 0.25981 rpy=3.1416 -1.0472 3.1416 -> xyz=0.3 0 0 rpy=3.1416 -1.0472 3.1416

Commit message: Added parallel leg config, fixing kinematics issue

File: src/res/flyhopper_mockup/urdf/flyhopper_mockup.urdf (robot description, URDF)
Before this commit: robot flyhopper_mockup, 3 links, 2 joints
Links:
- link Link 1: geometry collision mesh filename=package://../res/flyhopper_mockup/meshes/Link 1.STL; visual mesh filename=package://../res/flyhopper_mockup/meshes/Link 1.STL
- link Link 2: geometry collision mesh filename=package://../res/flyhopper_mockup/meshes/Link 2.STL; visual mesh filename=package://../res/flyhopper_mockup/meshes/Link 2.STL
- link base_link: geometry collision mesh filename=package://../res/flyhopper_mockup/meshes/base_link.STL; visual mesh filename=package://../res/flyhopper_mockup/meshes/base_link.STL

Commit message: Quick fix for URDF

File: src/res/flyhopper_mockup/urdf/flyhopper_mockup.urdf (robot description, URDF)
Before this commit: robot flyhopper_mockup, 3 links, 2 joints
Links:
- link base_link: geometry collision mesh filename=package://../res/flyhopper_mockup/meshes/base_link.STL; visual mesh filename=package://../res/flyhopper_mockup/meshes/base_link.STL
