Commit message: Rearranged directories, updated julia test code

File: res/flyhopper_mockup/urdf/flyhopper_mockup.urdf (robot description, URDF)
Before this commit: robot flyhopper_mockup, 3 links, 2 joints
Links:
- link Link 1: geometry collision mesh filename=package://../res/flyhopper_mockup/meshes/Link 1.stl; visual mesh filename=package://../res/flyhopper_mockup/meshes/Link 1.stl
- link Link 2: geometry collision mesh filename=package://../res/flyhopper_mockup/meshes/Link 2.stl; visual mesh filename=package://../res/flyhopper_mockup/meshes/Link 2.stl
- link base_link: geometry collision mesh filename=package://../../res/flyhopper_mockup/meshes/base_link.stl; visual mesh filename=package://../../res/flyhopper_mockup/meshes/base_link.stl

File: res/flyhopper_parallel/urdf/flyhopper_parallel.urdf (robot description, URDF)
Before this commit: robot flyhopper_parallel, 5 links, 4 joints
Links:
- link Link 1: geometry collision mesh filename=package://../../res/flyhopper_parallel/meshes/Link 1.STL; visual mesh filename=package://../../res/flyhopper_parallel/meshes/Link 1.STL
- link Link 2: geometry collision mesh filename=package://../../res/flyhopper_parallel/meshes/Link 2.STL; visual mesh filename=package://../../res/flyhopper_parallel/meshes/Link 2.STL
- link Link 3: geometry collision mesh filename=package://../../res/flyhopper_parallel/meshes/Link 3.STL; visual mesh filename=package://../../res/flyhopper_parallel/meshes/Link 3.STL
- link Link 4: geometry collision mesh filename=package://../../res/flyhopper_parallel/meshes/Link 4.STL; visual mesh filename=package://../../res/flyhopper_parallel/meshes/Link 4.STL
- link base_link: geometry collision mesh filename=package://../../res/flyhopper_parallel/meshes/base_link.STL; visual mesh filename=package://../../res/flyhopper_parallel/meshes/base_link.STL

Commit message: Updated serial_test_1

File: res/flyhopper_mockup/urdf/flyhopper_mockup.urdf (robot description, URDF)
Before this commit: robot flyhopper_mockup, 3 links, 2 joints
Links:
- link Link 1: geometry collision mesh filename=package://../../res/flyhopper_mockup/meshes/Link 1.stl; visual mesh filename=package://../../res/flyhopper_mockup/meshes/Link 1.stl
- link Link 2: geometry collision mesh filename=package://../../res/flyhopper_mockup/meshes/Link 2.stl; visual mesh filename=package://../../res/flyhopper_mockup/meshes/Link 2.stl

File: res/flyhopper_mockup/urdf/flyhopper_mockup_jl.urdf (robot description, URDF)
Before this commit: robot flyhopper_mockup, 3 links, 2 joints
Links:
- link Link 1: geometry collision mesh filename=../../res/flyhopper_mockup/meshes/Link 1.stl; visual mesh filename=../../res/flyhopper_mockup/meshes/Link 1.stl
- link Link 2: geometry collision mesh filename=../../res/flyhopper_mockup/meshes/Link 2.stl; visual mesh filename=../../res/flyhopper_mockup/meshes/Link 2.stl
