Commit message: Fixed issues with actuator model

File: res/flyhopper_mockup/urdf_5kg/flyhopper_mockup.urdf (robot description, URDF)
Before this commit: robot flyhopper_mockup, 3 links, 2 joints
Links:
- link Link 1: geometry collision mesh filename=package://../../res/flyhopper_mockup/meshes/Link 1.stl; visual mesh filename=package://../../res/flyhopper_mockup/meshes/Link 1.stl
- link Link 2: geometry collision mesh filename=package://../../res/flyhopper_mockup/meshes/Link 2.stl; visual mesh filename=package://../../res/flyhopper_mockup/meshes/Link 2.stl
- link base_link: geometry collision mesh filename=package://../../res/flyhopper_mockup/meshes/base_link.stl; visual mesh filename=package://../../res/flyhopper_mockup/meshes/base_link.stl
Joints:
- joint Joint 2: limit lower=-3.14 upper=3.14 effort=0 velocity=0 -> lower=-1.92 upper=3.14 effort=0 velocity=0

File: res/flyhopper_mockup/urdf_5kg/flyhopper_mockup_jl.urdf (robot description, URDF)
Before this commit: robot flyhopper_mockup, 3 links, 2 joints
Links:
- link Link 1: geometry collision mesh filename=../../res/flyhopper_mockup/meshes/Link 1.stl; visual mesh filename=../../res/flyhopper_mockup/meshes/Link 1.stl
- link Link 2: geometry collision mesh filename=../../res/flyhopper_mockup/meshes/Link 2.stl; visual mesh filename=../../res/flyhopper_mockup/meshes/Link 2.stl
- link base_link: mass 10 -> 5; geometry collision mesh filename=../../res/flyhopper_mockup/meshes/base_link.stl; visual mesh filename=../../res/flyhopper_mockup/meshes/base_link.stl
