Commit message: Rewriting leg_parallel to use lagrangian formulation

File: res/flyhopper_robot/urdf/flyhopper_robot_jl.urdf (robot description, URDF)
Before this commit: robot flyhopper_robot, 5 links, 4 joints
Links:
- link Link 0: geometry collision mesh filename=package://../../res/flyhopper_robot/meshes/Link 0.STL; visual mesh filename=package://../../res/flyhopper_robot/meshes/Link 0.STL
- link Link 1: geometry collision mesh filename=package://../../res/flyhopper_robot/meshes/Link 1.STL; visual mesh filename=package://../../res/flyhopper_robot/meshes/Link 1.STL
- link Link 2: geometry collision mesh filename=package://../../res/flyhopper_robot/meshes/Link 2.STL; visual mesh filename=package://../../res/flyhopper_robot/meshes/Link 2.STL
- link Link 3: geometry collision mesh filename=package://../../res/flyhopper_robot/meshes/Link 3.STL; visual mesh filename=package://../../res/flyhopper_robot/meshes/Link 3.STL
- link base_link: geometry collision mesh filename=package://../../res/flyhopper_robot/meshes/base_link.STL; visual mesh filename=package://../../res/flyhopper_robot/meshes/base_link.STL
