Commit message: Simplified state machine by removing redundant crouch state, added adaptive PID tuning for contact vs non-contact

File: res/flyhopper_rw/urdf/flyhopper_rw.urdf (robot description, URDF)
Before this commit: robot flyhopper_rw, 7 links, 6 joints
Joints:
- joint Joint 1: limit lower=-0.7597 upper=0.8295 effort=0 velocity=0 -> lower=-0.7597 upper=1.8295 effort=0 velocity=0
- joint Joint 3: limit lower=-0.8295 upper=0.7597 effort=0 velocity=0 -> lower=-1.8295 upper=0.7597 effort=0 velocity=0
