Commit message: Updated rev05 urdf files

File: res/hopper_rev05/urdf/hopper_rev05.urdf (robot description, URDF)
Before this commit: robot hopper_rev05, 8 links, 7 joints
Links:
- link Link 0: mass 0.256385566504166 -> 0.256385566503952
- link Link 1: mass 0.0631473819780344 -> 0.0631473819780702
- link Link 2: mass 0.288845046277992 -> 0.288845046277886
- link Link 3: mass 0.124857603952318 -> 0.12485760282637
- link base_link: mass 5.49365283282163 -> 5.59607837933863
- link rw1: mass 0.715641175076261 -> 0.715641175076257
- link rwz: mass 0.480621066769277 -> 0.377854494953541
Joints:
- joint Joint 0: origin xyz=0 0 0 rpy=0 0.523598775598299 0 -> xyz=0 0 0 rpy=0 0.5235987755983 0
- joint Joint 1: origin xyz=0.1 0 0 rpy=-3.14159265358979 1.0768315178335 -3.14159265358979 -> xyz=0.0999999999999999 0 0 rpy=-3.14159265358979 1.0768315178335 -3.14159265358979
- joint Joint 2: origin xyz=0 0 0 rpy=3.14159265358979 0.553232742319404 3.14159265358979 -> xyz=0 0 0 rpy=3.14159265358979 0.553232742319403 -3.14159265358979
- joint joint_rw0: origin xyz=0.0620132647100509 -0.14725367593953 0 rpy=3.03065856040946 0 -0.785398163397452 -> xyz=0.0620132647100599 -0.147253675939521 0 rpy=3.03065856040946 0 -0.785398163397452
- joint joint_rw1: origin xyz=0.062013264710069 0.147253675939512 0 rpy=-0.0304329711040608 0 0.785398163397453 -> xyz=0.063525686232125 0.148766097461586 0 rpy=-0.0304329711040608 0 0.785398163397453
- joint joint_rwz: origin xyz=-0.0666999999999999 0 0.1015 rpy=0 0 -1.5707963267949 -> xyz=-0.076 0 0.0991000000000001 rpy=0 0 -2.35619449019233
