Commit message: Removed legacy parallel, serial, and belt models, revamped plotting

File: res/hopper_cmg/urdf/hopper_cmg.urdf (robot description, URDF)
Before this commit: robot hopper_cmg, 14 links, 13 joints
Links:
- link Link 3: mass 0.124857600403456 -> 0.124857600224648
- link base_link: mass 4.33217212737128 -> 4.33217212044982
- link gimbal1: mass 0.145059160959023 -> 0.145059160959022
- link gimbal3: mass 0.145059160100867 -> 0.145059160100868
- link rw0: mass 0.0987820774247233 -> 0.0987820774247236
- link rw1: mass 0.0987820774247232 -> 0.0987820774247234
- link rw2: mass 0.0987820774247234 -> 0.0987820774247233
- link rwz: mass 0.377854494953541 -> 0.377854494953542
Joints:
- joint joint_gimbal0: axis 0.707106781186545 0 -0.70710678118655 -> 0 0 1; limit (none) -> lower=0 upper=0 effort=0 velocity=0; origin xyz=0.0200818325856985 -0.143506009999232 0.0469999999999983 rpy=1.5707963267949 0 0.785398163397444 -> xyz=0.020082 -0.14351 0.047 rpy=1.5708 0 0.7854; type fixed -> revolute
- joint joint_gimbal1: axis -0.707106781186544 0 0.707106781186551 -> 0 0 1; limit (none) -> lower=0 upper=0 effort=0 velocity=0; origin xyz=0.104934646328085 -0.058653196256847 0.0469999999999984 rpy=1.5707963267949 0 0.785398163397444 -> xyz=0.10493 -0.058653 0.047 rpy=1.5708 0 0.7854; type fixed -> revolute
- joint joint_gimbal2: axis 0 0 0 -> 0 0 1; limit (none) -> lower=0 upper=0 effort=0 velocity=0; origin xyz=0.104934646328084 0.058653196256847 0.0470000000000001 rpy=1.5707963267949 0 2.35619449019235 -> xyz=0.10493 0.058653 0.047 rpy=1.5708 0 2.3562; type fixed -> revolute
- joint joint_gimbal3: axis 0 0 0 -> 0 0 1; limit (none) -> lower=0 upper=0 effort=0 velocity=0; origin xyz=0.0200818325856976 0.143506009999232 0.047 rpy=1.5707963267949 0 2.35619449019235 -> xyz=0.020082 0.14351 0.047 rpy=1.5708 0 2.3562; type fixed -> revolute
- joint joint_rw3: origin xyz=0 0 0 rpy=-0.018598308001901 0 1.5707963267949 -> xyz=0 0 0 rpy=-0.018598 0 1.5708
- joint joint_rwz: origin xyz=-0.076 0 0.0991000000000001 rpy=0 0 -2.35619449019233 -> xyz=-0.076 0 0.0991 rpy=0 0 -2.3562

Commit message: Troubleshooting cmg issues

File: res/hopper_cmg/urdf/hopper_cmg.urdf (robot description, URDF)
Before this commit: robot hopper_cmg, 14 links, 13 joints
Links:
- link Link 2: mass 0.288845046277886 -> 0.288845047026487
- link Link 3: mass 0.124857600224648 -> 0.124857602987161
- link base_link: mass 4.33217212044982 -> 4.33217212032757
- link gimbal2: mass 0.145059153810549 -> 0.14505915381055
- link gimbal3: mass 0.145059160100868 -> 0.145059160100867
- link rw0: mass 0.0987820774247236 -> 0.109706994641609
- link rw1: mass 0.0987820774247234 -> 0.109706994641609
- link rw2: mass 0.0987820774247233 -> 0.109706994641609
- link rw3: mass 0.0987820774247234 -> 0.109706994641609
- link rwz: mass 0.377854494953542 -> 0.377854494953543
Joints:
- joint joint_gimbal0: origin xyz=0.020082 -0.14351 0.047 rpy=1.5708 0 0.7854 -> xyz=0.0434163563648536 -0.166840533778391 0.047 rpy=1.5707963267949 0 0.785398163397444
- joint joint_gimbal1: limit lower=0 upper=0 effort=0 velocity=0 -> lower=-1.57 upper=1.57 effort=0 velocity=0; origin xyz=0.10493 -0.058653 0.047 rpy=1.5708 0 0.7854 -> xyz=0.12827 -0.081988 0.047 rpy=1.5708 0 0.7854
- joint joint_gimbal2: limit lower=0 upper=0 effort=0 velocity=0 -> lower=-1.57 upper=1.57 effort=0 velocity=0; origin xyz=0.10493 0.058653 0.047 rpy=1.5708 0 2.3562 -> xyz=0.12827 0.081988 0.047 rpy=1.5708 0 2.3562
- joint joint_gimbal3: limit lower=0 upper=0 effort=0 velocity=0 -> lower=-1.57 upper=1.57 effort=0 velocity=0; origin xyz=0.020082 0.14351 0.047 rpy=1.5708 0 2.3562 -> xyz=0.043416 0.16684 0.047 rpy=1.5708 0 2.3562
- joint joint_rw0: axis 0 1 0 -> 0 0 -1; origin xyz=0 0 0 rpy=0 -0.834873615401156 3.14159265358979 -> xyz=0 0.0157238798738165 -0.033 rpy=1.5707963267949 0.73592271139374 3.14159265358979
- joint joint_rw1: axis 0 1 0 -> 0 0 -1; origin xyz=0 0 0 rpy=0 0.0185983080019021 3.14159265358979 -> xyz=0 0.0157238798738165 -0.033 rpy=-1.57079632679489 1.55219801879299 0
- joint joint_rw2: axis 0 1 0 -> 0 0 -1; origin xyz=0 0 0 rpy=0 -0.834873615401156 3.14159265358979 -> xyz=0 0.0157238798738165 -0.0329999999999979 rpy=1.5707963267949 0.73592271139374 3.14159265358979
- joint joint_rw3: axis -1 0 0 -> 0 0 -1; origin xyz=0 0 0 rpy=-0.018598 0 1.5708 -> xyz=0 0.0157238798738165 -0.033 rpy=-1.57079632679489 1.55219801879299 0
- joint joint_rwz: origin xyz=-0.076 0 0.0991 rpy=0 0 -2.3562 -> xyz=-0.076 0 0.0991000000000001 rpy=0 0 -2.35619449019233
