Commit message: Updated rev08 model with accurate inertias, re-tuning

File: res/hopper_rev08/urdf/hopper_rev08.urdf (robot description, URDF)
Before this commit: robot hopper_rev08, 8 links, 7 joints
Links:
- link Link 0: mass 0.586954605797748 -> 0.58695463086016
- link Link 1: mass 0.0631473819780334 -> 0.0631473819780293
- link Link 2: mass 0.619414111352979 -> 0.61941411063406
- link Link 3: mass 0.124857600438339 -> 0.124857597355403
- link base_link: mass 4.51400070312395 -> 4.38051667799002
- link rw0: mass 0.711638774644899 -> 0.712386930815601
- link rw1: mass 0.711638774351903 -> 0.712386930742353
- link rwz: mass 0.356354012275079 -> 0.356354012275082
Joints:
- joint Joint 0: origin xyz=0 0 0 rpy=0 0.5236 0 -> xyz=0 0 0 rpy=0 0.523598775598322 0
- joint Joint 1: origin xyz=0.1 0 0 rpy=3.1416 1.0768 3.1416 -> xyz=0.0999999999999984 0 0 rpy=3.14159265358979 1.07683151783354 3.14159265358979
- joint Joint 2: origin xyz=0 0 0 rpy=3.1416 0.55323 3.1416 -> xyz=0 0 0 rpy=3.14159265358979 0.553232742319411 3.14159265358979
- joint Joint 3: origin xyz=0.27 0 0 rpy=-3.1416 -1.0768 3.1416 -> xyz=0.270000000042221 0 0 rpy=-3.14159265358979 -1.0768315174382 3.14159265358979
- joint joint_rw0: origin xyz=0.056569 -0.1372 0 rpy=3.1416 0 -0.7854 -> xyz=0.0565685424949263 -0.137195959492894 0 rpy=3.14159265358979 0 -0.785398163397437
- joint joint_rw1: origin xyz=0.056569 0.1372 0 rpy=0 0 0.7854 -> xyz=0.0565685424949229 0.137195959492894 0 rpy=0 0 0.785398163397453
